File: Hardware/SlugMesh.kicad_sch (KiCad schematic)
At the start: 2 parts, among them U1 STM32WLE5CCUx, U2 SKY66122

Commit message: chips throwup
Parts:
- added FL1: B2671, Filter:Filter_1109-5_1.1x0.9mm, symbol Filter:SAFFB942MFM0F0A
- added U3: BALFHB-WL-02D3, parts:CSPG8_STM, symbol parts:BALFHB-WL-02D3
- added U4: STUSB4500QTR, Package_DFN_QFN:QFN-24-1EP_4x4mm_P0.5mm_EP2.7x2.7mm, symbol Interface_USB:STUSB4500QTR
- added U5: BQ25887, Package_DFN_QFN:VQFN-24-1EP_4x4mm_P0.5mm_EP2.5x2.5mm, symbol Battery_Management:BQ25887
- added U6: CP2102N-Axx-xQFN20, Package_DFN_QFN:SiliconLabs_QFN-20-1EP_3x3mm_P0.5mm_EP1.8x1.8mm, symbol Interface_USB:CP2102N-Axx-xQFN20
Connections:
- new net: FL1.2, FL1.5
- new net: U4.10 (GND), U4.25 (GND)
- new net: U6.12 (GND), U6.21 (GND), U6.3 (GND)
- new net: U5.13 (BAT), U5.14 (BAT)
- new net: U5.15 (SNS), U5.16 (SNS)
- new net: U5.17 (SW), U5.18 (SW)
- new net: U5.19 (GND), U5.20 (GND)
- new net: U5.21 (PMID), U5.22 (PMID)
Other:
- moved on the sheet: U1, U2
